File: analog hat.kicad_pcb (KiCad board)
At the start: 2 copper layers, 40.6 x 28.7 mm, 12 parts, among them J4 Conn_01x06, J5 Conn_01x10, J6 Conn_01x10, U1 MCP1541-TO, U3 MCP4922-ESL, U4 MCP3204

Commit message: Fix ICs placement
Parts:
- moved C2 3.20 mm to (153.7, 148.8)
- moved U1 3.07 mm to (155.0, 152.5)
- moved C1 3.04 mm to (149.7, 152.5)
- moved C8 0.20 mm to (141.8, 136.6)
- moved U4 0.20 mm to (159.4, 139.8)
Routing:
- net /VREF: track 37.7 -> 35.7 mm
